File: hardware/dwm1000_arduino/indicators.kicad_sch (KiCad schematic)
At the start: 12 parts

Commit message: finixh schematic and first pass layout
Parts:
- C1: footprint (none) -> Capacitor_SMD:C_0805_2012Metric_Pad1.18x1.45mm_HandSolder; DigiKey (none) -> 445-12654-6-ND
- D1, D2: footprint (none) -> LED_THT:LED_D5.0mm-4_RGB; DigiKey (none) -> 1528-1959-ND
- D3, D4, D5: footprint (none) -> LED_SMD:LED_0805_2012Metric_Pad1.15x1.40mm_HandSolder; DigiKey (none) -> 475-2560-6-ND
- D6: value SFDLED -> RXOKLED; footprint (none) -> LED_SMD:LED_0805_2012Metric_Pad1.15x1.40mm_HandSolder; DigiKey (none) -> 475-2560-6-ND
- JP1: footprint (none) -> Jumper:SolderJumper-2_P1.3mm_Open_RoundedPad1.0x1.5mm
- R2, R3, R4, R5: footprint (none) -> Resistor_SMD:R_0805_2012Metric_Pad1.20x1.40mm_HandSolder; DigiKey (none) -> RMCF0805JT200RDKR-ND

Commit message: start rev 2 of the dwm board
Parts:
- removed C1: 10uF, Capacitor_SMD:C_0805_2012Metric_Pad1.18x1.45mm_HandSolder, symbol Device:C_Small
- removed D1, D2: NeoPixel_THT, LED_THT:LED_D5.0mm-4_RGB, symbol LED:NeoPixel_THT
- removed D3: TXLED, LED_SMD:LED_0805_2012Metric_Pad1.15x1.40mm_HandSolder, symbol Device:LED_Small
- removed D4: RXLED, LED_SMD:LED_0805_2012Metric_Pad1.15x1.40mm_HandSolder, symbol Device:LED_Small
- removed D5: SFDLED, LED_SMD:LED_0805_2012Metric_Pad1.15x1.40mm_HandSolder, symbol Device:LED_Small
- removed D6: RXOKLED, LED_SMD:LED_0805_2012Metric_Pad1.15x1.40mm_HandSolder, symbol Device:LED_Small
- removed JP1: SKIP_NEOS, Jumper:SolderJumper-2_P1.3mm_Open_RoundedPad1.0x1.5mm, symbol Jumper:SolderJumper_2_Open
- removed R2, R3, R4, R5: 200, Resistor_SMD:R_0805_2012Metric_Pad1.20x1.40mm_HandSolder, symbol Device:R_Small
Other:
- note removed: "Bypass cap for neopixels"
