File: hardware/dwm1000_arduino/power.kicad_sch (KiCad schematic)
At the start: 5 parts

Commit message: rev 2 pcb schematic
Parts:
- added C10, C12: 1uF, symbol Device:C_Small
- added C14: 4.7uF, symbol Device:C_Small
- added F4: 500mA, Fuse:Fuse_1206_3216Metric_Pad1.42x1.75mm_HandSolder, symbol Device:Fuse_Small
- added U3: MIC5239-3.3YM, Package_SO:SOIC-8_3.9x4.9mm_P1.27mm, symbol Regulator_Linear:MIC5365-3.3YC5
- gave numbers to parts that had none: 5
Connections:
- net +3V3: now also F4.2
- net +5V: now also C10.1, U3.1 (EN), U3.3 (VIN)
- net GND: now also C10.2, C12.2, C14.2, U3.5 (GND), U3.6 (GND), U3.7 (GND), U3.8 (GND)
- new net: C12.1, C14.1, F4.1, U3.4 (VOUT)
Other:
- moved on the sheet: C11, C13, C9, F3, U2

Commit message: finish layout
Parts:
- C10, C11, C12, C13, C14, C9: footprint (none) -> Capacitor_SMD:C_0805_2012Metric_Pad1.18x1.45mm_HandSolder
Connections:
- net 3V3_UNFUSED: now reaches C12.1, C14.1, F4.1, U3.4 (VOUT)
- net 5V_UNFUSED: now reaches C11.1, C13.1, F3.1, U2.4 (VOUT)
Other:
- note added: "Input: 5V-20V Output: 3V3 @ 500mA"
- note added: "Place near pin 3"
- note added: "Place near pin 4"
- note removed: "TODO: Spec 3V3 LDO"
Changed lines of the file:
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@@
     (stroke (width 0) (type default) (color 0 0 0 0))
   )
+  (text "Input: 5V-20V\nOutput: 3V3 @ 500mA" (at 160.02 160.02 0)
+    (effects (font (size 1.27 1.27)) (justify left bottom))
+  )
   (text "Input: 5V-20V\nOutput: 5V @ 500mA" (at 160.02 116.84 0)
     (effects (font (size 1.27 1.27)) (justify left bottom))
   )
-  (text "TODO: Spec 3V3 LDO" (at 144.78 124.46 0)
+  (text "Place near pin 3" (at 115.57 144.78 0)
+    (effects (font (size 1.27 1.27)) (justify left bottom))
+  )
+  (text "Place near pin 3" (at 115.57 100.33 0)
+    (effects (font (size 1.27 1.27)) (justify left bottom))
+  )
+  (text "Place near pin 4" (at 189.23 100.33 0)
+    (effects (font (size 1.27 1.27)) (justify left bottom))
+  )
+  (text "Place near pin 4" (at 189.23 144.78 0)
+    (effects (font (size 1.27 1.27)) (justify left bottom))
+  )
+  (label "3V3_UNFUSED" (at 177.8 134.62 0)
+    (effects (font (size 1.27 1.27)) (justify left bottom))
+  )
+  (label "5V_UNFUSED" (at 177.8 90.17 0)
     (effects (font (size 1.27 1.27)) (justify left bottom))
   )
@@
       (effects (font (size 1.27 1.27)) (justify left))
     )
-    (property "Footprint" "" (id 2) (at 185.42 95.25 0)
+    (property "Footprint" "Capacitor_SMD:C_0805_2012Metric_Pad1.18x1.45mm_HandSolder" (id 2) (at 185.42 95.25 0)
       (effects (font (size 1.27 1.27)) hide)
     )
@@
       (effects (font (size 1.27 1.27)) (justify left))
     )
-    (property "Footprint" "" (id 2) (at 176.53 139.7 0)
+    (property "Footprint" "Capacitor_SMD:C_0805_2012Metric_Pad1.18x1.45mm_HandSolder" (id 2) (at 176.53 139.7 0)
       (effects (font (size 1.27 1.27)) hide)
     )
@@
       (effects (font (size 1.27 1.27)) (justify left))
     )
-    (property "Footprint" "" (id 2) (at 135.89 139.7 0)
+    (property "Footprint" "Capacitor_SMD:C_0805_2012Metric_Pad1.18x1.45mm_HandSolder" (id 2) (at 135.89 139.7 0)
       (effects (font (size 1.27 1.27)) hide)
     )
@@
       (effects (font (size 1.27 1.27)) (justify left))
     )
-    (property "Footprint" "" (id 2) (at 135.89 95.25 0)
+    (property "Footprint" "Capacitor_SMD:C_0805_2012Metric_Pad1.18x1.45mm_HandSolder" (id 2) (at 135.89 95.25 0)
       (effects (font (size 1.27 1.27)) hide)
     )
@@
       (effects (font (size 1.27 1.27)) (justify left))
     )
-    (property "Footprint" "" (id 2) (at 176.53 95.25 0)
+    (property "Footprint" "Capacitor_SMD:C_0805_2012Metric_Pad1.18x1.45mm_HandSolder" (id 2) (at 176.53 95.25 0)
       (effects (font (size 1.27 1.27)) hide)
     )
@@
       (effects (font (size 1.27 1.27)) (justify left))
     )
-    (property "Footprint" "" (id 2) (at 185.42 139.7 0)
-      (effects (font (size 1.27 1.27)) hide)
-    )
+    (property "Footprint" "Capacitor_SMD:C_0805_2012Metric_Pad1.18x1.45mm_HandSolder" (id 2) (at 185.42 139.7 0)
+      (effects (font (size 1.27 1.27)) hide)
+    )
